Commit message: add sample launchs

File: urdf/skid_steer_unitree_example.urdf (robot description, URDF)
Before this commit: robot quadro_unitree_example, 5 links, 4 joints
Links:
- removed link none1
- removed link none2
- removed link none3
- removed link none4
- removed link unitree
- added link base_link
- added link fl_wheel
- added link fr_wheel
- added link rl_wheel
- added link rr_wheel
Joints:
- removed joint unitree_joint1
- removed joint unitree_joint2
- removed joint unitree_joint3
- removed joint unitree_joint4
- added joint fl_wheel_joint: type continuous, parent base_link, child fl_wheel
- added joint fr_wheel_joint: type continuous, parent base_link, child fr_wheel
- added joint rl_wheel_joint: type continuous, parent base_link, child rl_wheel
- added joint rr_wheel_joint: type continuous, parent base_link, child rr_wheel
