Commit message: more organized example

File: examples/single_unitree/description/ros2_control.xacro (robot description, xacro)
@@ -1,14 +1,10 @@
-<robot name="single_unitree_example">
-    <link name="unitree" />
-    <joint name="unitree_joint" type="continuous">
-        <parent link="unitree" />
-        <child link="none" />
-    </joint>
-    <link name="none" />
-    <!-- -->
+<?xml version="1.0"?>
+<robot>
     <ros2_control name="LayeredHardware" type="system">
         <hardware>
             <plugin>layered_hardware/LayeredHardware</plugin>
             <param name="layers">
+                - name: monitor_layer
+                  type: layered_hardware/MonitorLayer
                 - name: joint_limits_layer
                   type: layered_hardware/JointLimitsLayer
@@ -20,28 +16,28 @@
             <param name="unitree_actuator_layer">
                 actuators:
-                    unitree_actuator:
+                    axis_unitree:
                         id: 0
                         motor_type: GO-M8010-6
                         operating_mode_map:
-                            unitree_joint/position: position
-                            unitree_joint/velocity: velocity
-                            unitree_joint/effort: torque
+                            axis/position: position
+                            axis/velocity: velocity
+                            axis/effort: torque
             </param>
         </hardware>
-        <joint name="unitree_joint">
+        <joint name="axis">
             <command_interface name="position">
-                <param name="min">-10</param>
-                <param name="max">10</param>
+                <!-- <param name="min">-1.0</param> -->
+                <!-- <param name="max">1.0</param> -->
             </command_interface>
-            <command_interface name="velocity">
-            </command_interface>
-            <command_interface name="effort">
-            </command_interface>
+            <command_interface name="velocity" />
+            <command_interface name="effort" />
             <state_interface name="position"/>
+            <state_interface name="velocity"/>
+            <state_interface name="effort"/>
         </joint>
-        <transmission name="unitree_trans">
+        <transmission name="axis_trans">
             <plugin>transmission_interface/SimpleTransmission</plugin>
-            <actuator name="unitree_actuator" role="unitree_actuator"/>
-            <joint name="unitree_joint" role="unitree_joint">
+            <actuator name="axis_unitree" role="axis_unitree"/>
+            <joint name="axis" role="axis">
                 <mechanical_reduction>1.0</mechanical_reduction>
                 <offset>0.0</offset>

Commit message: more natural roles for transmission components

File: examples/single_unitree/description/ros2_control.xacro (robot description, xacro)
@@ -38,6 +38,6 @@
         <transmission name="axis_trans">
             <plugin>transmission_interface/SimpleTransmission</plugin>
-            <actuator name="axis_unitree" role="axis_unitree"/>
-            <joint name="axis" role="axis">
+            <actuator name="axis_unitree" role="actuator"/>
+            <joint name="axis" role="joint">
                 <mechanical_reduction>1.0</mechanical_reduction>
                 <offset>0.0</offset>
